Commit message: Add new option for homework wit limits

File: urdf/IRB14000.urdf (robot description, URDF)
Before this commit: robot irf, 15 links, 14 joints
Links:
- link 1R: mass 0.962860384395944 -> 0
- link 2L: mass 1.41046348706547 -> 1.41045545917515
- link 2R: mass 1.41050001295053 -> 1.41053215466353
- link 3L: mass 0.71081197360719 -> 0.710813617750004
- link 3R: mass 0.718728305997546 -> 0.718724825102295
- link 4L: mass 1.18080238238893 -> 1.18079192762883
- link 4R: mass 1.18078971547547 -> 1.18080282713249
- link 5L: mass 0.34341459827255 -> 0.343419516713393
- link 5R: mass 0.343463913186024 -> 0.343456193438038
- link 6L: mass 0.465742953606289 -> 0.465741945501003
- link 6R: mass 0.470288404060638 -> 0.47028030766964
- link 7L: mass 0.0309416727783666 -> 0.0309424125499957
- link 7R: mass 0.0416752390294235 -> 0.0416752660026345
- link base_link: mass 10.2333776403801 -> 10.233377644213
Joints:
- joint 01L: limit (none) -> lower=-0.9654 upper=0.9654 effort=0 velocity=0; origin xyz=0.35042 -0.50866 0.31984 rpy=0.78956 0.2634 -0.42471 -> xyz=-0.0057377 0.047589 0.38069 rpy=-0.65168 -0.39991 -0.28481; type continuous -> revolute
- joint 01R: axis 0.8138 -0.34202 0.46985 -> 0.813797681347725 -0.3420201433221 0.469846310398407; limit (none) -> lower=-0.9654 upper=0.9654 effort=0 velocity=0; origin xyz=0.43511 -0.55756 0.25939 rpy=2.2247 -0.24632 -0.34724 -> xyz=-0.0905970285494174 -0.0119241865590318 0.331693781179444 rpy=0.661249391678768 -0.407079130841712 0.287099256033239; type continuous -> revolute
- joint 12L: limit (none) -> lower=0.8914 upper=2.06 effort=0 velocity=0; origin xyz=0.20488 0.11189 0.14434 rpy=-1.3437 -0.48353 2.2404 -> xyz=0.12122 0.076728 0.096038 rpy=-1.4686 -0.326 2.4813; type continuous -> revolute
- joint 12R: axis 0.10678 -0.70672 -0.69939 -> 0.106777674127034 -0.706717031145236 -0.699392283484229; limit (none) -> lower=-2.06 upper=-0.8914 effort=0 velocity=0; origin xyz=0.12019 -0.076297 0.095446 rpy=1.3853 -0.44056 -2.3146 -> xyz=0.20607785829111 -0.112392243464449 0.145031664519265 rpy=1.47821664003411 -0.309277896876161 -2.50290546025724; type continuous -> revolute
- joint 23L: limit (none) -> lower=-0.9654 upper=0.9654 effort=0 velocity=0; origin xyz=0.13409 0.031233 0.050602 rpy=1.4041 -0.068337 0.87651 -> xyz=0.015536 -0.018591 -0.017844 rpy=-0.00079928 -0.00033614 -0.00046138; type continuous -> revolute
- joint 23R: axis 0.8138 -0.34202 0.46985 -> 0.813797681351336 -0.34202014335914 0.469846310365191; limit (none) -> lower=-0.9654 upper=0.9654 effort=0 velocity=0; origin xyz=0 0.01 0 rpy=-1.3757 -0.053924 -0.86134 -> xyz=0.0915183890471042 -0.0120186622456074 0.0275466493971784 rpy=-0.039448450188403 0.0160500394071166 -0.0229876231436337; type continuous -> revolute
- joint 34L: limit (none) -> lower=-1.0192 upper=0.77 effort=0 velocity=0; origin xyz=0.11095 0.011822 0.028884 rpy=-0.058551 0.50311 -0.52682 -> xyz=0.2295 0.061646 0.09733 rpy=-0.041579 0.46212 -0.47621; type continuous -> revolute
- joint 34R: axis 0.10678 -0.70672 -0.69939 -> 0.106777674130013 -0.706717031141072 -0.699392283487982; limit (none) -> lower=-0.64 upper=1.3 effort=0 velocity=0; origin xyz=0.23263 -0.058464 0.094592 rpy=0.01936 0.39352 0.39696 -> xyz=0.15236620264851 -0.0292295290745919 0.0527977154113355 rpy=0.0717762948550856 0.530708904391656 0.562616525117697; type continuous -> revolute
- joint 45L: axis 0.57125 -0.61933 -0.5386 -> 0.571254638611826 -0.619332914863809 -0.538604565920834; limit (none) -> lower=-1.6616 upper=1.6616 effort=0 velocity=0; origin xyz=0.15495 -0.11841 -0.095989 rpy=1.8182 0.12991 -1.7527 -> xyz=0.115196356607472 -0.0753070608732511 -0.0585084857542666 rpy=-0.0171887920517601 0.0189406911212764 0.0161881718975502; type continuous -> revolute
- joint 45R: axis 0.57125 0.61933 -0.5386 -> 0.571254638611776 0.619332914864763 -0.53860456591979; limit (none) -> lower=-1.6616 upper=1.6616 effort=0 velocity=0; origin xyz=0.13312 0.11448 -0.061036 rpy=-1.8973 0.24174 1.8253 -> xyz=0.0713634822125091 0.0277850981332976 -0.0171808807510679 rpy=0.00444066455296555 0.00483466417264907 -0.00418566420803987; type continuous -> revolute
- joint 56L: axis 0.10678 0.70672 -0.69939 -> 0.106777674107038 0.706717031146258 -0.69939228348625; limit (none) -> lower=-0.5042 upper=0.7907 effort=0 velocity=0; origin xyz=0.0074198 -0.041101 -0.040398 rpy=3.5585E-05 0.30278 -0.29968 -> xyz=0.0471728145210148 -0.0841993484533884 -0.0778791980350019 rpy=-0.0103654032994117 0.357314140710582 -0.357295616611069; type continuous -> revolute
- joint 56R: axis 0.10678 -0.70672 -0.69939 -> 0.10677767414999 -0.706717031153939 -0.69939228347193; limit (none) -> lower=-0.5042 upper=0.7907 effort=0 velocity=0; origin xyz=0.023092 0.058092 -0.055175 rpy=-0.0096611 0.21444 0.21021 -> xyz=0.087412497123785 0.127825707411432 -0.115818980607626 rpy=-0.00730342604387015 0.0604081215420703 0.0593475847532015; type continuous -> revolute
- joint 67L: axis 0.57125 -0.61933 -0.5386 -> 0.571254638614449 -0.619332914870399 -0.538604565910475; limit (none) -> lower=-1.3121 upper=1.3121 effort=0 velocity=0; origin xyz=0.022079 0.0099413 0.011986 rpy=-0.16152 0.20366 0.1503 -> xyz=0.022079315069325 0.00994126089859926 0.0119864580985115 rpy=1.31235264605213 -0.294889504789811 -1.27042178310482; type continuous -> revolute
- joint 67R: axis 0.57125 0.61933 -0.5386 -> 0.571254638614754 0.619332914870736 -0.538604565909764; limit (none) -> lower=-1.3121 upper=1.3121 effort=0 velocity=0; origin xyz=0.022079 -0.0099413 0.011986 rpy=0.19164 0.24837 -0.17775 -> xyz=0.0220793150687765 -0.00994126090174002 0.0119864580948938 rpy=0.666032477367434 1.15259582967801 -0.511862372677926; type continuous -> revolute

Commit message: gazebo main.launch and urdf - change

File: urdf/IRB14000.urdf (robot description, URDF)
Before this commit: robot irf, 15 links, 14 joints
Links:
- link 1R: mass 0 -> 0.926

Commit message: urdf change

File: urdf/IRB14000.urdf (robot description, URDF)
Before this commit: robot irf, 15 links, 14 joints
Joints:
- joint 67L: limit lower=-1.3121 upper=1.3121 effort=0 velocity=0 -> lower=-1.3121 upper=1.3121 effort=0 velocity=0.0

Commit message: Change in urdf inertia for 1R

File: urdf/IRB14000.urdf (robot description, URDF)
Before this commit: robot irf, 15 links, 14 joints
Links:
- link 1R: mass 0.926 -> 0.92686
